Commit message: remap topic names

File: rover_bot/urdf/rover_bot.xacro (robot description, xacro)
@@ -14,4 +14,5 @@
     <color rgba="0 1 0 1"/>
   </material>
+  <!-- robot -->
   <xacro:include filename="$(find rover_bot)/urdf/rover_bot.gazebo" />
   <link name="robot_footprint"></link>
@@ -205,4 +206,12 @@
         <parent link="chassis"/>
     </joint>
+    <!-- rgbd camera -->
+    <link name="camera_rgbd_frame"/>
+    <!-- camera rgbd joint -->
+    <joint name="camera_rgbd_joint" type="fixed">
+      <origin xyz="0 0 0" rpy="-1.5707 0 -1.5707"/>
+      <child link="camera_rgbd_frame"/>
+      <parent link="camera"/>
+    </joint>
     <!-- Laser Rangefinder link -->
     <link name="hokuyo">
